Commit message: risolto imu (sasi sei un coglione)

File: src/pkg/rover_description_pkg/urdf/imu.urdf (robot description, URDF)
Before this commit: robot imu, 1 links, 1 joints
Links:
- removed link imu_link
Joints:
- removed joint imu_to_payload

File: src/pkg/rover_description_pkg/urdf/rover.xacro (robot description, xacro)
@@ -5,4 +5,5 @@
 <xacro:include filename="$(find rover_description_pkg)/urdf/utilities.xacro"/>
 <xacro:include filename="$(find rover_description_pkg)/urdf/rover_gazebo.xacro"/>
+<xacro:include filename="$(find rover_description_pkg)/urdf/imu.urdf" />
 <xacro:arg name="is_sim" default="true"/>
 <xacro:arg name="namespace" default="/" />
@@ -15,4 +16,5 @@
   <xacro:camera_gazebo camera_base_frame="camera_link" camera_topic="camera" camera_info_topic="camera_info" prefix="$(arg prefix)"/>
 </xacro:if>
+<xacro:imu_macro prefix="$(arg prefix)"/>
 <!-- if it is in simulation -->
     <!--

File: src/pkg/rover_description_pkg/urdf/rover_macro.xacro (robot description, xacro)
@@ -23,5 +23,4 @@
   <xacro:property name="wheel_mass" value="1.25" />
   <xacro:property name="payload_z_offset" value="0.096" />
-  <!-- <xacro:include filename="$(find rover_description_pkg)/urdf/imu.urdf"/> -->
   <!-- Macro del telaio -->
   <xacro:macro name="rover_base_frame" params="prefix">
