Commit message: risolto imu e cameraù

File: src/pkg/rover_description_pkg/urdf/rover.xacro (robot description, xacro)
@@ -5,4 +5,5 @@
 <xacro:include filename="$(find rover_description_pkg)/urdf/utilities.xacro"/>
 <xacro:include filename="$(find rover_description_pkg)/urdf/rover_gazebo.xacro"/>
+<xacro:include filename="$(find rover_description_pkg)/urdf/imu.urdf" />
 <xacro:include filename="$(find rover_description_pkg)/urdf/imu.urdf" />
 <xacro:arg name="is_sim" default="true"/>
@@ -13,7 +14,5 @@
 <xacro:gazebo_diff_drive_controller left_joint="diff_drive_l_joint" right_joint="diff_drive_r_joint" prefix= "$(arg prefix)" namespace="$(arg namespace)" />
 <xacro:gazebo_wheel_contact prefix="(arg prefix)"/>
-<xacro:if value="$(eval prefix == 'master')">
-  <xacro:camera_gazebo camera_base_frame="camera_link" camera_topic="camera" camera_info_topic="camera_info" prefix="$(arg prefix)"/>
-</xacro:if>
+<xacro:camera_gazebo camera_base_frame="camera_link" camera_topic="camera" camera_info_topic="camera_info" prefix="$(arg prefix)"/>
 <xacro:imu_macro prefix="$(arg prefix)"/>
 <!-- if it is in simulation -->

File: src/pkg/rover_description_pkg/urdf/rover_gazebo.xacro (robot description, xacro)
@@ -113,10 +113,10 @@
         <origin xyz="0 0 0" rpy="0 0 0"/>
     </xacro:sensor_d435i>  -->
-    <joint name="camera_to_payload" type="fixed">
+    <joint name="${prefix}_camera_to_payload" type="fixed">
         <origin xyz="0.02 0 ${1 -0.129 - total_height}" rpy="0 0 0"/>
         <parent link="${prefix}_payload_link"/>
-        <child link="${camera_base_frame}"/>
-    </joint>
-    <link name="${camera_base_frame}">
+        <child link="${prefix}_${camera_base_frame}"/>
+    </joint>
+    <link name="${prefix}_${camera_base_frame}">
         <visual>
         <origin xyz="0 0 0" rpy="1.57 0 1.57"/>
@@ -132,35 +132,35 @@
         </collision>
     </link>
-  <joint name="camera_rgb_joint" type="fixed">
+  <joint name="${prefix}_camera_rgb_joint" type="fixed">
     <origin xyz="0.005 0.018 0.013" rpy="0 0 0"/>
-    <parent link="${camera_base_frame}"/>
-    <child link="camera_rgb_frame"/>
-  </joint>
-  <link name="camera_rgb_frame"/>
-  <joint name="camera_rgb_optical_joint" type="fixed">
+    <parent link="${prefix}_${camera_base_frame}"/>
+    <child link="${prefix}_camera_rgb_frame"/>
+  </joint>
+  <link name="${prefix}_camera_rgb_frame"/>
+  <joint name="${prefix}_camera_rgb_optical_joint" type="fixed">
     <origin xyz="0 0 0" rpy="-1.57 0 -1.57"/>
-    <parent link="camera_rgb_frame"/>
-    <child link="camera_rgb_optical_frame"/>
-  </joint>
-  <link name="camera_rgb_optical_frame"/>
-  <joint name="camera_depth_joint" type="fixed">
+    <parent link="${prefix}_camera_rgb_frame"/>
+    <child link="${prefix}_camera_rgb_optical_frame"/>
+  </joint>
+  <link name="${prefix}_camera_rgb_optical_frame"/>
+  <joint name="${prefix}_camera_depth_joint" type="fixed">
     <origin xyz="0.005 0.028 0.013" rpy="0 0 0"/>
-    <parent link="${camera_base_frame}"/>
-    <child link="camera_depth_frame"/>
-  </joint>
-  <link name="camera_depth_frame"/>
-  <joint name="camera_depth_optical_joint" type="fixed">
+    <parent link="${prefix}_${camera_base_frame}"/>
+    <child link="${prefix}_camera_depth_frame"/>
+  </joint>
+  <link name="${prefix}_camera_depth_frame"/>
+  <joint name="${prefix}_camera_depth_optical_joint" type="fixed">
     <origin xyz="0 0 0" rpy="0 0 0"/>
-    <parent link="camera_depth_frame"/>
-    <child link="camera_depth_optical_frame"/>
-  </joint>
-  <link name="camera_depth_optical_frame"/>
-    <gazebo reference="${camera_base_frame}">
+    <parent link="${prefix}_camera_depth_frame"/>
+    <child link="${prefix}_camera_depth_optical_frame"/>
+  </joint>
+  <link name="${prefix}_camera_depth_optical_frame"/>
+    <gazebo reference="${prefix}_${camera_base_frame}">
         <sensor name="d435_color" type="camera">
-            <topic>color/image_raw</topic>
-            <ignition_frame_id>rover/camera_link</ignition_frame_id>
-            <gz_frame_id>rover/camera_link</gz_frame_id>
+            <topic>${prefix}/color/image_raw</topic>
+            <ignition_frame_id>${prefix}/camera_link</ignition_frame_id>
+            <gz_frame_id>${prefix}/camera_link</gz_frame_id>
             <camera name="d435">
-                <camera_info_topic>color/camera_info</camera_info_topic>
+                <camera_info_topic>${prefix}/color/camera_info</camera_info_topic>
                 <horizontal_fov>1.21126</horizontal_fov>
 				<image>
@@ -187,10 +187,10 @@
 			<update_rate>10</update_rate>
 			<visualize>0</visualize>
-			<topic>depth/image_raw</topic>
-            <ignition_frame_id>rover/camera_depth_optical_frame</ignition_frame_id>
+			<topic>${prefix}/depth/image_raw</topic>
+            <ignition_frame_id>${prefix}/camera_depth_optical_frame</ignition_frame_id>
 			<pose>0 0.0175 0.5125 0 -0 0</pose>
 			<camera name="d435">
-                <point_cloud_topic>depth/color/points</point_cloud_topic>
-                <camera_info_topic>depth/camera_info</camera_info_topic>
+                <point_cloud_topic>${prefix}/depth/color/points</point_cloud_topic>
+                <camera_info_topic>${prefix}/depth/camera_info</camera_info_topic>
 				<horizontal_fov>1.48702</horizontal_fov>
 				<image>
@@ -210,9 +210,11 @@
 		</sensor>
     </gazebo>
-    <gazebo>
-        <plugin filename="libignition-gazebo-sensors-system.so" name="ignition::gazebo::systems::Sensors">
-            <render_engine>ogre2</render_engine>
-        </plugin>
-    </gazebo>
+    <xacro:if value="$(eval prefix == 'master')">
+        <gazebo>
+            <plugin filename="libignition-gazebo-sensors-system.so" name="ignition::gazebo::systems::Sensors">
+                \<render_engine>ogre2</render_engine>
+            </plugin>
+        </gazebo>
+    </xacro:if>
 </xacro:macro>
     <!-- Gazebo Plugins -->

Commit message: TO DO: aggiungere slave con NAV2

File: src/pkg/rover_description_pkg/urdf/rover.xacro (robot description, xacro)
@@ -1,22 +1,19 @@
 <?xml version="1.0"?>
 <robot xmlns:xacro="http://www.ros.org/wiki/xacro" name="rover">
-<xacro:arg name="prefix" default=" " />
 <xacro:include filename="$(find rover_description_pkg)/urdf/rover_macro.xacro"/>
 <xacro:include filename="$(find rover_description_pkg)/urdf/utilities.xacro"/>
 <xacro:include filename="$(find rover_description_pkg)/urdf/rover_gazebo.xacro"/>
 <xacro:include filename="$(find rover_description_pkg)/urdf/imu.urdf" />
-<xacro:include filename="$(find rover_description_pkg)/urdf/imu.urdf" />
 <xacro:arg name="is_sim" default="true"/>
-<xacro:arg name="namespace" default="/" />
-<xacro:rover_base_frame prefix="$(arg prefix)"/>
-<xacro:lidar_gazebo_sensor laser_frame="lidar_link" laser_topic="scan" prefix="$(arg prefix)"/>
-<xacro:rover_wheels_sim left_joint="diff_drive_l_joint" right_joint="diff_drive_r_joint" prefix="$(arg prefix)"/>
-<xacro:gazebo_diff_drive_controller left_joint="diff_drive_l_joint" right_joint="diff_drive_r_joint" prefix= "$(arg prefix)" namespace="$(arg namespace)" />
-<xacro:gazebo_wheel_contact prefix="(arg prefix)"/>
-<xacro:camera_gazebo camera_base_frame="camera_link" camera_topic="camera" camera_info_topic="camera_info" prefix="$(arg prefix)"/>
-<xacro:imu_macro prefix="$(arg prefix)"/>
+<xacro:arg name="namespace" default="default"/>
+<link name="base_footprint">
+</link>
+<xacro:rover_base_frame parent_link="base_footprint"/>
 <!-- if it is in simulation -->
-    <!--
-    <xacro:camera_gazebo camera_base_frame="camera_link" camera_topic="camera" camera_info_topic="camera_info"/>
-     -->
+    <xacro:rover_wheels_sim left_joint="diff_drive_l_joint" right_joint="diff_drive_r_joint"/>
+    <xacro:gazebo_diff_drive_controller left_joint="diff_drive_l_joint" right_joint="diff_drive_r_joint" namespace="$(arg namespace)"/>
+    <xacro:gazebo_wheel_contact/>
+    <xacro:lidar_gazebo_sensor laser_frame="lidar_link" laser_topic="scan" namespace="$(arg namespace)"/>
+    <xacro:camera_gazebo camera_base_frame="camera_link" camera_topic="camera" camera_info_topic="camera_info" namespace="$(arg namespace)"/>
+<xacro:imu_macro namespace="$(arg namespace)"/>
 </robot>

File: src/pkg/rover_description_pkg/urdf/rover_gazebo.xacro (robot description, xacro)
@@ -1,6 +1,6 @@
 <?xml version="1.0"?>
 <robot xmlns:xacro="http://www.ros.org/wiki/xacro" name="rover_gazebo">
-<xacro:macro name="rover_wheels_sim" params="left_joint right_joint prefix">
-    <link name="${prefix}_fr_wheel_link">
+<xacro:macro name="rover_wheels_sim" params="left_joint right_joint">
+    <link name="fr_wheel_link">
         <visual>
             <origin xyz="0 0 0" rpy="-1.57 0 0" />
@@ -22,11 +22,11 @@
         <mu>5.0</mu>
     </link>
-    <joint name="${prefix}_fr_wheel_to_base" type="continuous">
-        <parent link="${prefix}_base_link"/>
-        <child link="${prefix}_fr_wheel_link"/>
+    <joint name="fr_wheel_to_base" type="continuous">
+        <parent link="base_link"/>
+        <child link="fr_wheel_link"/>
         <axis xyz="0 1 0"/>
         <origin xyz="${wheel_x_offset + front_flipper_x_offset} ${-wheel_y_offset} 0" rpy="0 0 0"/>
     </joint>
-    <link name="${prefix}_fl_wheel_link">
+    <link name="fl_wheel_link">
         <visual>
             <origin xyz="0 0 0" rpy="1.57 0 0" />
@@ -48,11 +48,11 @@
         <mu>5.0</mu>
     </link>
-    <joint name="${prefix}_fl_wheel_to_base" type="continuous">
-        <parent link="${prefix}_base_link"/>
-        <child link="${prefix}_fl_wheel_link"/>
+    <joint name="fl_wheel_to_base" type="continuous">
+        <parent link="base_link"/>
+        <child link="fl_wheel_link"/>
         <axis xyz="0 1 0"/>
         <origin xyz="${wheel_x_offset + front_flipper_x_offset} ${wheel_y_offset} 0" rpy="0 0 0"/>
     </joint>
-    <link name="${prefix}_rr_wheel_link">
+    <link name="rr_wheel_link">
         <visual>
             <origin xyz="0 0 0" rpy="1.57 0 3.1415" />
@@ -74,11 +74,11 @@
         <mu>5.0</mu>
     </link>
-    <joint name="${prefix}_rr_wheel_to_base" type="continuous">
-        <parent link="${prefix}_base_link"/>
-        <child link="${prefix}_rr_wheel_link"/>
+    <joint name="rr_wheel_to_base" type="continuous">
+        <parent link="base_link"/>
+        <child link="rr_wheel_link"/>
         <axis xyz="0 1 0"/>
         <origin xyz="${-wheel_x_offset} ${-wheel_y_offset} 0"/>
     </joint>
-    <link name="${prefix}_rl_wheel_link">
+    <link name="rl_wheel_link">
         <visual>
             <origin xyz="0 0 0" rpy="-1.57 0 3.1415" />
@@ -100,7 +100,7 @@
         <mu>5.0</mu>
     </link>
-    <joint name="${prefix}_rl_wheel_to_base" type="continuous">
-        <parent link="${prefix}_base_link"/>
-        <child link="${prefix}_rl_wheel_link"/>
+    <joint name="rl_wheel_to_base" type="continuous">
+        <parent link="base_link"/>
+        <child link="rl_wheel_link"/>
         <axis xyz="0 1 0"/>
         <origin xyz="${-wheel_x_offset} ${wheel_y_offset} 0"/>
@@ -108,15 +108,15 @@
 </xacro:macro>
 <!-- Camera -->
-<xacro:macro name="camera_gazebo" params="camera_base_frame camera_topic camera_info_topic prefix">
+<xacro:macro name="camera_gazebo" params="camera_base_frame camera_topic camera_info_topic namespace">
     <xacro:include filename="$(find realsense2_description)/urdf/_d435i.urdf.xacro"/>
     <!-- <xacro:sensor_d435i parent="${camera_base_frame}" use_nominal_extrinsics="true">
         <origin xyz="0 0 0" rpy="0 0 0"/>
     </xacro:sensor_d435i>  -->
-    <joint name="${prefix}_camera_to_payload" type="fixed">
+    <joint name="camera_to_payload" type="fixed">
         <origin xyz="0.02 0 ${1 -0.129 - total_height}" rpy="0 0 0"/>
-        <parent link="${prefix}_payload_link"/>
-        <child link="${prefix}_${camera_base_frame}"/>
-    </joint>
-    <link name="${prefix}_${camera_base_frame}">
+        <parent link="payload_link"/>
+        <child link="${camera_base_frame}"/>
+    </joint>
+    <link name="${camera_base_frame}">
         <visual>
         <origin xyz="0 0 0" rpy="1.57 0 1.57"/>
@@ -132,35 +132,35 @@
         </collision>
     </link>
-  <joint name="${prefix}_camera_rgb_joint" type="fixed">
+  <joint name="camera_rgb_joint" type="fixed">
     <origin xyz="0.005 0.018 0.013" rpy="0 0 0"/>
-    <parent link="${prefix}_${camera_base_frame}"/>
-    <child link="${prefix}_camera_rgb_frame"/>
-  </joint>
-  <link name="${prefix}_camera_rgb_frame"/>
-  <joint name="${prefix}_camera_rgb_optical_joint" type="fixed">
+    <parent link="${camera_base_frame}"/>
+    <child link="camera_rgb_frame"/>
+  </joint>
+  <link name="camera_rgb_frame"/>
+  <joint name="camera_rgb_optical_joint" type="fixed">
     <origin xyz="0 0 0" rpy="-1.57 0 -1.57"/>
-    <parent link="${prefix}_camera_rgb_frame"/>
-    <child link="${prefix}_camera_rgb_optical_frame"/>
-  </joint>
-  <link name="${prefix}_camera_rgb_optical_frame"/>
-  <joint name="${prefix}_camera_depth_joint" type="fixed">
+    <parent link="camera_rgb_frame"/>
+    <child link="camera_rgb_optical_frame"/>
+  </joint>
+  <link name="camera_rgb_optical_frame"/>
+  <joint name="camera_depth_joint" type="fixed">
     <origin xyz="0.005 0.028 0.013" rpy="0 0 0"/>
-    <parent link="${prefix}_${camera_base_frame}"/>
-    <child link="${prefix}_camera_depth_frame"/>
-  </joint>
-  <link name="${prefix}_camera_depth_frame"/>
-  <joint name="${prefix}_camera_depth_optical_joint" type="fixed">
+    <parent link="${camera_base_frame}"/>
+    <child link="camera_depth_frame"/>
+  </joint>
+  <link name="camera_depth_frame"/>
+  <joint name="camera_depth_optical_joint" type="fixed">
     <origin xyz="0 0 0" rpy="0 0 0"/>
-    <parent link="${prefix}_camera_depth_frame"/>
-    <child link="${prefix}_camera_depth_optical_frame"/>
-  </joint>
-  <link name="${prefix}_camera_depth_optical_frame"/>
-    <gazebo reference="${prefix}_${camera_base_frame}">
+    <parent link="camera_depth_frame"/>
+    <child link="camera_depth_optical_frame"/>
+  </joint>
+  <link name="camera_depth_optical_frame"/>
+    <gazebo reference="${camera_base_frame}">
         <sensor name="d435_color" type="camera">
-            <topic>${prefix}/color/image_raw</topic>
-            <ignition_frame_id>${prefix}/camera_link</ignition_frame_id>
-            <gz_frame_id>${prefix}/camera_link</gz_frame_id>
+            <!-- <topic>${namespace}/color/image_raw</topic>
+            <ignition_frame_id>${namespace}/camera_link</ignition_frame_id>
+            <gz_frame_id>${namespace}/camera_link</gz_frame_id> -->
             <camera name="d435">
-                <camera_info_topic>${prefix}/color/camera_info</camera_info_topic>
+                <!-- <camera_info_topic>${namespace}/color/camera_info</camera_info_topic> -->
                 <horizontal_fov>1.21126</horizontal_fov>
 				<image>
@@ -187,10 +187,10 @@
 			<update_rate>10</update_rate>
 			<visualize>0</visualize>
-			<topic>${prefix}/depth/image_raw</topic>
-            <ignition_frame_id>${prefix}/camera_depth_optical_frame</ignition_frame_id>
+			<!-- <topic>${namespace}/depth/image_raw</topic>
+            <ignition_frame_id>${namespace}/camera_depth_optical_frame</ignition_frame_id> -->
 			<pose>0 0.0175 0.5125 0 -0 0</pose>
 			<camera name="d435">
-                <point_cloud_topic>${prefix}/depth/color/points</point_cloud_topic>
-                <camera_info_topic>${prefix}/depth/camera_info</camera_info_topic>
+                <!-- <point_cloud_topic>${namespace}/depth/color/points</point_cloud_topic>
+                <camera_info_topic>${namespace}/depth/camera_info</camera_info_topic> -->
 				<horizontal_fov>1.48702</horizontal_fov>
 				<image>
@@ -210,5 +210,5 @@
 		</sensor>
     </gazebo>
-    <xacro:if value="$(eval prefix == 'master')">
+    <xacro:if value="$(eval namespace == 'master')">
         <gazebo>
             <plugin filename="libignition-gazebo-sensors-system.so" name="ignition::gazebo::systems::Sensors">
@@ -219,13 +219,13 @@
 </xacro:macro>
     <!-- Gazebo Plugins -->
-<xacro:macro name="gazebo_diff_drive_controller" params="left_joint right_joint namespace prefix">
+<xacro:macro name="gazebo_diff_drive_controller" params="left_joint right_joint namespace">
     <gazebo>
         <plugin name="ignition::gazebo::systems::DiffDrive" filename="ignition-gazebo-diff-drive-system">
             <num_wheel_pairs>2</num_wheel_pairs>
             <!-- Wheel Information -->
-            <left_joint>${prefix}_rl_wheel_to_base</left_joint>
-            <left_joint>${prefix}_fl_wheel_to_base</left_joint>
-            <right_joint>${prefix}_rr_wheel_to_base</right_joint>
-            <right_joint>${prefix}_fr_wheel_to_base</right_joint>
+            <left_joint>rl_wheel_to_base</left_joint>
+            <left_joint>fl_wheel_to_base</left_joint>
+            <right_joint>rr_wheel_to_base</right_joint>
+            <right_joint>fr_wheel_to_base</right_joint>
             <wheel_separation>0.37</wheel_separation>
             <wheel_radius>0.102</wheel_radius>
@@ -236,18 +236,18 @@
             <min_angular_acceleration>-4</min_angular_acceleration>
             <!-- Output -->
-            <frame_id>${namespace}odom</frame_id>
-            <child_frame_id>/${prefix}_base_link</child_frame_id>
+            <!-- <frame_id>/odom</frame_id>
+            <child_frame_id>/base_link</child_frame_id> -->
             <!-- Topics -->
-            <topic>/${namespace}cmd_vel</topic>
-            <odom_topic>/${namespace}odom/wheels</odom_topic>
-            <tf_topic>/${namespace}tf_gazebo</tf_topic>
+            <!-- <topic>/model/master/cmd_vel</topic>
+            <odom_topic>/odom/wheels</odom_topic>
+            <tf_topic>/tf_gazebo</tf_topic> -->
         </plugin>
         <plugin filename="ignition-gazebo-joint-state-publisher-system" name="ignition::gazebo::systems::JointStatePublisher">
-            <topic>/${namespace}joint_states</topic>
+            <!-- <topic>/model/master/joint_states</topic> -->
         </plugin>
     </gazebo>
 </xacro:macro>
-<xacro:macro name="gazebo_wheel_contact" params="prefix">
-    <gazebo reference="${prefix}_diff_wheel_left">
+<xacro:macro name="gazebo_wheel_contact">
+    <gazebo reference="diff_wheel_left">
         <mu1 value="1.0"/>
         <mu2 value="1.0"/>
@@ -256,5 +256,5 @@
         <fdir1 value="0 0 1"/>
     </gazebo>
-    <gazebo reference="${prefix}_diff_wheel_right">
+    <gazebo reference="diff_wheel_right">
         <mu1 value="1.0"/>
         <mu2 value="1.0"/>
@@ -263,26 +263,26 @@
         <fdir1 value="0 0 1"/>
     </gazebo>
-    <gazebo reference="${prefix}_collision_f_l">
-        <mu1 value="0.1"/>
-        <mu2 value="0.1"/>
-        <kp value="10000000.0"/>
-        <kd value="100.0"/>
-        <minDepth>0.001</minDepth>
-    </gazebo>
-    <gazebo reference="${prefix}_collision_f_r">
-        <mu1 value="0.1"/>
-        <mu2 value="0.1"/>
-        <kp value="10000000.0"/>
-        <kd value="100.0"/>
-        <minDepth>0.001</minDepth>
-    </gazebo>
-    <gazebo reference="${prefix}_collision_b_l">
-        <mu1 value="0.1"/>
-        <mu2 value="0.1"/>
-        <kp value="10000000.0"/>
-        <kd value="100.0"/>
-        <minDepth>0.001</minDepth>
-    </gazebo>
-    <gazebo reference="${prefix}_collision_b_r">
+    <gazebo reference="collision_f_l">
+        <mu1 value="0.1"/>
+        <mu2 value="0.1"/>
+        <kp value="10000000.0"/>
+        <kd value="100.0"/>
+        <minDepth>0.001</minDepth>
+    </gazebo>
+    <gazebo reference="collision_f_r">
+        <mu1 value="0.1"/>
+        <mu2 value="0.1"/>
+        <kp value="10000000.0"/>
+        <kd value="100.0"/>
+        <minDepth>0.001</minDepth>
+    </gazebo>
+    <gazebo reference="collision_b_l">
+        <mu1 value="0.1"/>
+        <mu2 value="0.1"/>
+        <kp value="10000000.0"/>
+        <kd value="100.0"/>
+        <minDepth>0.001</minDepth>
+    </gazebo>
+    <gazebo reference="collision_b_r">
         <mu1 value="0.1"/>
         <mu2 value="0.1"/>
