Commit message: TO DO: aggiungere slave con NAV2

File: src/pkg/rover_description_pkg/urdf/rover_macro.xacro (robot description, xacro)
@@ -1,140 +1,145 @@
 <?xml version="1.0"?>
 <robot xmlns:xacro="http://www.ros.org/wiki/xacro" name="rover_macro">
-  <!-- Proprietà rover -->
-  <xacro:property name="track_width" value="0.08"/>
-  <xacro:property name="total_width" value="0.4515"/>
-  <xacro:property name="total_length" value="0.422"/>
-  <xacro:property name="total_height" value="0.202"/>
-  <xacro:property name="chassis_width" value="0.241"/>
-  <xacro:property name="chassis_height" value="0.0785"/>
-  <xacro:property name="chassis_length" value="0.320"/>
-  <xacro:property name="track_distance" value="0.2915"/>
-  <xacro:property name="wheel_axes_distance" value="0.220"/>
-  <xacro:property name="wheel_collision_x" value="${total_length/2 - total_height/2 - 0.001}"/>
-  <xacro:property name="wheel_collision_y" value="${track_width}"/>
-  <xacro:property name="wheel_collision_z" value="${total_height - 0.02}"/>
-  <xacro:property name="rover_z_elev" value="${total_height/2 - chassis_height/2}"/>
-  <xacro:property name="collision_z_elev" value="${chassis_height/2}"/>
-  <xacro:property name="wheel_z_offset" value="0.020" />
-  <xacro:property name="wheel_x_offset" value="${wheel_axes_distance/2}" />
-  <xacro:property name="front_flipper_x_offset" value="-0.0035" />
-  <xacro:property name="wheel_y_offset" value="${(total_width-track_width)/2}" />
-  <xacro:property name="track_y_offset" value="0.11" />
-  <xacro:property name="wheel_mass" value="1.25" />
-  <xacro:property name="payload_z_offset" value="0.096" />
-  <!-- Macro del telaio -->
-  <xacro:macro name="rover_base_frame" params="prefix">
-    <link name="${prefix}_base_footprint"/>
-    <joint name="${prefix}_world_base_joint" type="fixed">
-      <parent link="${prefix}_base_footprint"/>
-      <child link="${prefix}_base_link"/>
-      <origin xyz="0.0 0.0 ${rover_z_elev}" rpy="0.0 0.0 0.0"/>
+        <!-- rover properties -->
+    <xacro:property name="track_width" value="0.08"/>
+    <xacro:property name="total_width" value="0.4515"/>
+    <xacro:property name="total_length" value="0.422"/>
+    <xacro:property name="total_height" value="0.202"/>
+    <xacro:property name="chassis_width" value="0.241"/>
+    <xacro:property name="chassis_height" value="0.0785"/>
+    <xacro:property name="chassis_length" value="0.320"/>
+    <xacro:property name="track_distance" value="0.2915"/>
+    <xacro:property name="wheel_axes_distance" value="0.220"/>
+    <xacro:property name="wheel_collision_x" value="${total_length/2 - total_height/2 - 0.001}"/>
+    <xacro:property name="wheel_collision_y" value="${track_width}"/>
+    <xacro:property name="wheel_collision_z" value="${total_height - 0.02}"/>
+    <xacro:property name="rover_z_elev" value="${total_height/2 - chassis_height/2}"/>
+    <xacro:property name="collision_z_elev" value="${chassis_height/2}"/>
+    <!-- Robot Parameters -->
+    <xacro:property name="wheel_z_offset" value="0.020" />
+    <xacro:property name="wheel_x_offset" value="${wheel_axes_distance/2}" />
+    <xacro:property name="front_flipper_x_offset" value="-0.0035" />
+    <xacro:property name="wheel_y_offset" value="${(total_width-track_width)/2}" />
+    <xacro:property name="track_y_offset" value="0.11" />
+    <xacro:property name="wheel_mass" value="1.25" />
+    <xacro:property name="payload_z_offset" value="0.096" />
+    <!-- <xacro:include filename="$(find rover_description_pkg)/urdf/imu.urdf" /> -->
+    <xacro:macro name="rover_base_frame" params="parent_link">
+        <joint name="world_base_joint" type="fixed">
+            <parent link="${parent_link}"/>
+            <child link="base_link"/>
+            <origin xyz="0.0 0.0 ${rover_z_elev}" rpy="0.0 0.0 0.0"/>
+        </joint>
+        <link name="base_link">
+            <visual>
+                <origin xyz="0 0 -0.035" rpy="0 0 0" />
+                <geometry>
+                    <mesh filename="file://$(find rover_description_pkg)/meshes/prisma_rover.stl" scale="0.001 0.001 0.001"/>
+                </geometry>
+                <material name="grey">
+                    <color rgba="0.2350821 0.2106182 0.2557221 1.0"/>
+                </material>
+            </visual>
+            <inertial>
+                <origin xyz="0.0 0.0 0.0" rpy="0.0 0.0 0.0"/>
+                <mass value="10.0"/>
+                <!-- the x coefficient is a pezzotto to avoid rocking movement of the rover -->
+                <xacro:box_inertia m="10.0" x="${total_length}" y="${total_width}" z="${total_height}"/>
+            </inertial>
+            <collision>
+                <origin xyz="0.0 0.0 ${collision_z_elev}" rpy="0.0 0.0 0.0"/>
+                <geometry>
+                    <box size="${total_length} ${total_width - 2*track_width} ${total_height - 0.1}"/>
+                </geometry>
+            </collision>
+        </link>
+        <link name="pole_link">
+            <collision>
+            <origin xyz="0.0 0.0 0.0" rpy="0 0 0"/>
+                <geometry>
+                    <cylinder radius="0.0125" length="${1.1-2*total_height}"/>
+                </geometry>
+            </collision>
+        </link>
+    </xacro:macro>
+    <link name="payload_link">
+        <collision>
+            <origin xyz="-0.1 0.0 0.04" rpy="0 0 0" />
+            <geometry>
+                <box size="${total_length/4} ${total_width -4.5*track_width} 0.04"/>
+            </geometry>
+        </collision>
+        <inertial>
+            <origin xyz="-0.01 0 0" rpy="0 0 0"/>
+            <mass value="2.95" />
+            <inertia ixx="0.018398" ixy="0.0"  ixz="0.0" iyy="0.04064" iyz="0.0" izz="0.05396" />
+        </inertial>
+    </link>
+    <joint name="payload_to_base" type="fixed">
+        <parent link="base_link"/>
+        <child link="payload_link"/>
+        <origin xyz="0 0 0.14"/>
     </joint>
-    <link name="${prefix}_base_link">
-      <visual>
-        <origin xyz="0 0 -0.035" rpy="0 0 0"/>
-        <geometry>
-          <mesh filename="file://$(find rover_description_pkg)/meshes/prisma_rover.stl" scale="0.001 0.001 0.001"/>
-        </geometry>
-        <material name="grey">
-          <color rgba="0.2350821 0.2106182 0.2557221 1.0"/>
-        </material>
-      </visual>
-      <inertial>
-        <origin xyz="0.0 0.0 0.0" rpy="0.0 0.0 0.0"/>
-        <mass value="10.0"/>
-        <xacro:box_inertia m="10.0" x="${total_length}" y="${total_width}" z="${total_height}"/>
-      </inertial>
-      <collision>
-        <origin xyz="0.0 0.0 ${collision_z_elev}" rpy="0.0 0.0 0.0"/>
-        <geometry>
-          <box size="${total_length} ${total_width - 2*track_width} ${total_height - 0.1}"/>
-        </geometry>
-      </collision>
-    </link>
-    <link name="${prefix}_pole_link">
-      <collision>
-        <origin xyz="0.0 0.0 0.0" rpy="0 0 0"/>
-        <geometry>
-          <cylinder radius="0.0125" length="${1.1-2*total_height}"/>
-        </geometry>
-      </collision>
-    </link>
-    <link name="${prefix}_payload_link">
-      <collision>
-        <origin xyz="-0.1 0.0 0.04" rpy="0 0 0"/>
-        <geometry>
-          <box size="${total_length/4} ${total_width -4.5*track_width} 0.04"/>
-        </geometry>
-      </collision>
-      <inertial>
-        <origin xyz="-0.01 0 0" rpy="0 0 0"/>
-        <mass value="2.95"/>
-        <inertia ixx="0.018398" ixy="0.0" ixz="0.0" iyy="0.04064" iyz="0.0" izz="0.05396"/>
-      </inertial>
-    </link>
-    <joint name="${prefix}_payload_to_base" type="fixed">
-      <parent link="${prefix}_base_link"/>
-      <child link="${prefix}_payload_link"/>
-      <origin xyz="0 0 0.14"/>
+    <joint name="pole_to_payload" type="fixed">
+        <origin xyz="0 0 ${0.4 - total_height/2}" rpy="0 0 0"/>
+        <parent link="payload_link"/>
+        <child link="pole_link"/>
     </joint>
-    <joint name="${prefix}_pole_to_payload" type="fixed">
-      <origin xyz="0 0 ${0.4 - total_height/2}" rpy="0 0 0"/>
-      <parent link="${prefix}_payload_link"/>
-      <child link="${prefix}_pole_link"/>
-    </joint>
-  </xacro:macro>
-  <!-- LIDAR Macro -->
-  <xacro:macro name="lidar_gazebo_sensor" params="laser_frame laser_topic prefix">
-    <joint name="${prefix}_lidar_to_payload" type="fixed">
-      <parent link="${prefix}_payload_link"/>
-      <child link="${prefix}_${laser_frame}"/>
-      <origin xyz="0.075 0 -0.01" rpy="0.0 0.0 3.1415"/>
-    </joint>
-    <link name="${prefix}_${laser_frame}">
-      <visual>
-        <origin xyz="0 0 0" rpy="-1.57 0.0 3.1415"/>
-        <geometry>
-          <mesh filename="file://$(find rover_description_pkg)/meshes/rplidar_s2.dae"/>
-        </geometry>
-      </visual>
-      <collision>
-        <origin xyz="0 0 0" rpy="0 0 3.1415"/>
-        <geometry>
-          <cylinder radius="0.04" length="0.15"/>
-        </geometry>
-      </collision>
-    </link>
-    <gazebo reference="${prefix}_${laser_frame}">
-      <sensor name="gpu_lidar" type="gpu_lidar">
-        <pose>0 0 0 0 0 0</pose>
-        <topic>${laser_topic}</topic>
-        <ignition_frame_id>${laser_frame}</ignition_frame_id>
-        <gz_frame_id>${laser_frame}</gz_frame_id>
-        <update_rate>10</update_rate>
-        <lidar>
-          <scan>
-            <horizontal>
-              <samples>640</samples>
-              <resolution>1</resolution>
-              <min_angle>-3.14159</min_angle>
-              <max_angle>3.14159</max_angle>
-            </horizontal>
-            <vertical>
-              <samples>1</samples>
-              <resolution>1</resolution>
-              <min_angle>0.0</min_angle>
-              <max_angle>0.0</max_angle>
-            </vertical>
-          </scan>
-          <range>
-            <min>0.23</min>
-            <max>10.0</max>
-            <resolution>0.01</resolution>
-          </range>
-        </lidar>
-        <visualize>true</visualize>
-      </sensor>
+<xacro:macro name="lidar_gazebo_sensor" params="laser_frame laser_topic namespace">
+        <joint name="lidar_to_payload" type="fixed">
+            <parent link="payload_link"/>
+            <child link="${laser_frame}"/>
+            <origin xyz="0.075 0 -0.01" rpy="0.0 0.0 3.1415"/>
+        </joint>
+        <link name="${laser_frame}">
+            <visual>
+                <origin xyz="0 0 0" rpy="-1.57 0.0 3.1415"/>
+                <geometry>
+                    <mesh filename="file://$(find rover_description_pkg)/meshes/rplidar_s2.dae"/>
+                </geometry>
+            </visual>
+            <collision>
+                <origin xyz="0 0 0" rpy="0 0 3.1415"/>
+                <geometry>
+                    <cylinder radius="0.04" length="0.15"/>
+                </geometry>
+            </collision>
+        </link>
+        <gazebo reference="${laser_frame}">
+        <sensor name='gpu_lidar' type='gpu_lidar'>
+            <pose>0 0 0 0 0 0</pose>
+            <!-- <topic>/${laser_topic}</topic> -->
+            <ignition_frame_id>${namespace}/lidar_link</ignition_frame_id>
+            <gz_frame_id>${namespace}/lidar_link</gz_frame_id>
+            <update_rate>10</update_rate>
+            <lidar>
+                <scan>
+                <horizontal>
+                    <samples>640</samples>
+                    <resolution>1</resolution>
+                    <min_angle>-3.14159</min_angle>
+                    <max_angle>3.14159</max_angle>
+                </horizontal>
+                <vertical>
+                    <samples>1</samples>
+                    <resolution>1</resolution>
+                    <min_angle>0.0</min_angle>
+                    <max_angle>0.0</max_angle>
+                </vertical>
+                </scan>
+                <range>
+                <min>0.23</min>
+                <max>10.0</max>
+                <resolution>0.01</resolution>
+                </range>
+            </lidar>
+            <visualize>true</visualize>
+        </sensor>
     </gazebo>
-  </xacro:macro>
+    <!-- <gazebo>
+        <plugin filename="libignition-gazebo-sensors-system.so" name="ignition::gazebo::systems::Sensors">
+            <render_engine>ogre2</render_engine>
+        </plugin>
+    </gazebo> -->
+    </xacro:macro>
 </robot>
